File: KiCad/vssk.kicad_pcb (KiCad board)
At the start: 2 copper layers, 395 x 90.2 mm, 0 parts

Commit message: placed switch footprints
Parts:
- added C1: 10uF, keeb:C_0805_2012Metric, F.Cu at (50.8, 292.1)
- added C2: .1uF, keeb:C_0805_2012Metric, F.Cu at (68.4, 292.1)
- added C3: .1uF, keeb:C_0805_2012Metric, F.Cu at (81.7, 292.1)
- added C4: .1uF, keeb:C_0805_2012Metric, F.Cu at (55.2, 292.1)
- added C5: 22pf, keeb:C_0805_2012Metric, F.Cu at (59.6, 292.1)
- added C6: 22pf, keeb:C_0805_2012Metric, F.Cu at (64.0, 292.1)
- added C7: .1uF, keeb:C_0805_2012Metric, F.Cu at (42.0, 292.1)
- added C8: 1uF, keeb:C_0805_2012Metric, F.Cu at (77.3, 292.1)
- added D1: BAV70, Package_TO_SOT_SMD:SOT-23, F.Cu at (140.8, 287.8)
- added D10: BAV70, Package_TO_SOT_SMD:SOT-23, F.Cu at (47.6, 288.4)
- added D11: BAV70, Package_TO_SOT_SMD:SOT-23, F.Cu at (309.5, 145.1)
- added D12: BAV70, Package_TO_SOT_SMD:SOT-23, F.Cu at (228.7, 130.0)
- added D13: BAV70, Package_TO_SOT_SMD:SOT-23, F.Cu at (135.9, 287.8)
- added D14: BAV70, Package_TO_SOT_SMD:SOT-23, F.Cu at (140.5, 292.2)
- added D15: BAV70, Package_TO_SOT_SMD:SOT-23, F.Cu at (145.4, 292.2)
- added D16: BAV70, Package_TO_SOT_SMD:SOT-23, F.Cu at (164.9, 287.8)
- added D17: BAV70, Package_TO_SOT_SMD:SOT-23, F.Cu at (150.3, 292.2)
- added D18: BAV70, Package_TO_SOT_SMD:SOT-23, F.Cu at (76.9, 288.4)
- added D19: BAV70, Package_TO_SOT_SMD:SOT-23, F.Cu at (219.0, 174.8)
- added D2: BAV70, Package_TO_SOT_SMD:SOT-23, F.Cu at (57.4, 288.4)
- added D20: BAV70, Package_TO_SOT_SMD:SOT-23, F.Cu at (86.7, 288.4)
- added D21: BAV70, Package_TO_SOT_SMD:SOT-23, F.Cu at (62.3, 288.4)
- added D22: BAV70, Package_TO_SOT_SMD:SOT-23, F.Cu at (169.8, 287.8)
- added D23: BAV70, Package_TO_SOT_SMD:SOT-23, F.Cu at (219.0, 179.3)
- added D24: BAV70, Package_TO_SOT_SMD:SOT-23, F.Cu at (145.7, 287.8)
- added D25: BAV70, Package_TO_SOT_SMD:SOT-23, F.Cu at (81.8, 288.4)
- added D26: BAV70, Package_TO_SOT_SMD:SOT-23, F.Cu at (219.0, 165.9)
- added D27: BAV70, Package_TO_SOT_SMD:SOT-23, F.Cu at (125.8, 288.4)
- added D28: BAV70, Package_TO_SOT_SMD:SOT-23, F.Cu at (67.2, 288.4)
- added D29: BAV70, Package_TO_SOT_SMD:SOT-23, F.Cu at (228.7, 134.4)
- added D3: BAV70, Package_TO_SOT_SMD:SOT-23, F.Cu at (155.2, 292.2)
- added D30: BAV70, Package_TO_SOT_SMD:SOT-23, F.Cu at (52.5, 288.4)
- added D31: BAV70, Package_TO_SOT_SMD:SOT-23, F.Cu at (130.7, 292.2)
- added D32: BAV70, Package_TO_SOT_SMD:SOT-23, F.Cu at (72.0, 288.4)
- added D33: BAV70, Package_TO_SOT_SMD:SOT-23, F.Cu at (96.5, 288.4)
- added D34: BAV70, Package_TO_SOT_SMD:SOT-23, F.Cu at (271.2, 185.5)
- added D35: BAV70, Package_TO_SOT_SMD:SOT-23, F.Cu at (131.0, 287.8)
- added D36: BAV70, Package_TO_SOT_SMD:SOT-23, F.Cu at (228.7, 138.9)
- added D37: BAV70, Package_TO_SOT_SMD:SOT-23, F.Cu at (150.6, 287.8)
- added D38: BAV70, Package_TO_SOT_SMD:SOT-23, F.Cu at (228.7, 125.5)
- added D39: BAV70, Package_TO_SOT_SMD:SOT-23, F.Cu at (111.2, 288.4)
- added D4: BAV70, Package_TO_SOT_SMD:SOT-23, F.Cu at (219.0, 170.4)
- added D40: BAV70, Package_TO_SOT_SMD:SOT-23, F.Cu at (106.3, 288.4)
- added D41: BAV70, Package_TO_SOT_SMD:SOT-23, F.Cu at (101.4, 288.4)
- added D42: BAV70, Package_TO_SOT_SMD:SOT-23, F.Cu at (91.6, 288.4)
- added D43: BAV70, Package_TO_SOT_SMD:SOT-23, F.Cu at (164.9, 292.2)
- added D44: BAV70, Package_TO_SOT_SMD:SOT-23, F.Cu at (160.1, 287.8)
- added D45: BAV70, Package_TO_SOT_SMD:SOT-23, F.Cu at (120.9, 288.4)
- added D46: BAV70, Package_TO_SOT_SMD:SOT-23, F.Cu at (160.1, 292.2)
- added D5: BAV70, Package_TO_SOT_SMD:SOT-23, F.Cu at (37.8, 288.4)
- added D6: BAV70, Package_TO_SOT_SMD:SOT-23, F.Cu at (309.5, 149.5)
- added D7: BAV70, Package_TO_SOT_SMD:SOT-23, F.Cu at (42.7, 288.4)
- added D8: BAV70, Package_TO_SOT_SMD:SOT-23, F.Cu at (135.6, 292.2)
- added D9: BAV70, Package_TO_SOT_SMD:SOT-23, F.Cu at (116.0, 288.4)
- added J1: Conn_01x04, keeb:JST-SR-4, F.Cu at (31.5, 292.2)
- added JP1: Jumper_2_Bridged, keeb:ResetJumper, F.Cu at (115.0, 160.2)
- added R1: 22, keeb:R_0805_2012Metric, F.Cu at (113.0, 163.3)
- added R2: 22, keeb:R_0805_2012Metric, F.Cu at (37.6, 292.1)
- added R3: 10k, keeb:R_0805_2012Metric, F.Cu at (72.8, 292.1)
- added R4: 10k, keeb:R_0805_2012Metric, F.Cu at (46.4, 292.1)
- added SW1: M1, FancyHybridPrints:MX-1U-NoLED, F.Cu at (9.55, 9.75)
- added SW10: M10, FancyHybridPrints:MX-1U-NoLED, F.Cu at (28.6, 86.0)
- added SW11: `, FancyHybridPrints:MX-1U-NoLED, F.Cu at (57.2, 9.75)
- added SW12: Tab, FancyHybridPrints:MX-1.5U-NoLED, F.Cu at (61.9, 28.8)
- added SW13: Stepped Caps, FancyHybridPrints:MX-1.25U-NoLED, F.Cu at (59.6, 47.9)
- added SW14: Capslock, FancyHybridPrints:MX-1.75U-NoLED, F.Cu at (64.3, 47.9)
- added SW15: 2.25u Shift, FancyHybridPrints:MX-2.25U-NoLED, F.Cu at (69.1, 66.9)
- added SW16: 1.25u Shift, FancyHybridPrints:MX-1.25U-NoLED, F.Cu at (59.6, 66.9)
- added SW17: Ctrl, FancyHybridPrints:MX-1.5U-NoLED, F.Cu at (61.9, 86.0)
- added SW18: 1, FancyHybridPrints:MX-1U-NoLED, F.Cu at (76.2, 9.75)
- added SW19: Q, FancyHybridPrints:MX-1U-NoLED, F.Cu at (85.8, 28.8)
- added SW2: M3, FancyHybridPrints:MX-1U-NoLED, F.Cu at (9.55, 28.8)
- added SW20: \, FancyHybridPrints:MX-1U-NoLED, F.Cu at (81.0, 66.9)
- added SW21: 2, FancyHybridPrints:MX-1U-NoLED, F.Cu at (95.3, 9.75)
- added SW22: W, FancyHybridPrints:MX-1U-NoLED, F.Cu at (104.8, 28.8)
- added SW23: A, FancyHybridPrints:MX-1U-NoLED, F.Cu at (90.5, 47.9)
- added SW24: Z, FancyHybridPrints:MX-1U-NoLED, F.Cu at (100.0, 66.9)
- added SW25: Alt, FancyHybridPrints:MX-1.5U-NoLED, F.Cu at (109.6, 86.0)
- added SW26: 3, FancyHybridPrints:MX-1U-NoLED, F.Cu at (114.3, 9.75)
- added SW27: E, FancyHybridPrints:MX-1U-NoLED, F.Cu at (123.8, 28.8)
- added SW28: S, FancyHybridPrints:MX-1U-NoLED, F.Cu at (109.6, 47.9)
- added SW29: X, FancyHybridPrints:MX-1U-NoLED, F.Cu at (119.1, 66.9)
- added SW3: M5, FancyHybridPrints:MX-1U-NoLED, F.Cu at (9.55, 47.9)
- added SW30: 4, FancyHybridPrints:MX-1U-NoLED, F.Cu at (133.4, 9.75)
- added SW31: R, FancyHybridPrints:MX-1U-NoLED, F.Cu at (142.9, 28.8)
- added SW32: D, FancyHybridPrints:MX-1U-NoLED, F.Cu at (128.6, 47.9)
- added SW33: C, FancyHybridPrints:MX-1U-NoLED, F.Cu at (138.1, 66.9)
- added SW34: 5, FancyHybridPrints:MX-1U-NoLED, F.Cu at (152.4, 9.75)
- added SW35: T, FancyHybridPrints:MX-1U-NoLED, F.Cu at (161.9, 28.8)
- added SW36: F, FancyHybridPrints:MX-1U-NoLED, F.Cu at (147.7, 47.9)
- added SW37: V, FancyHybridPrints:MX-1U-NoLED, F.Cu at (157.2, 66.9)
- added SW38: 6, FancyHybridPrints:MX-1U-NoLED, F.Cu at (171.5, 9.75)
- added SW39: Y, FancyHybridPrints:MX-1U-NoLED, F.Cu at (181.0, 28.8)
- added SW4: M7, FancyHybridPrints:MX-1U-NoLED, F.Cu at (9.55, 66.9)
- added SW40: G, FancyHybridPrints:MX-1U-NoLED, F.Cu at (166.7, 47.9)
- added SW41: B, FancyHybridPrints:MX-1U-NoLED, F.Cu at (176.2, 66.9)
- added SW42: 7, FancyHybridPrints:MX-1U-NoLED, F.Cu at (190.5, 9.75)
- added SW43: U, FancyHybridPrints:MX-1U-NoLED, F.Cu at (200.1, 28.8)
- added SW44: H, FancyHybridPrints:MX-1U-NoLED, F.Cu at (185.8, 47.9)
- added SW45: N, FancyHybridPrints:MX-1U-NoLED, F.Cu at (195.3, 66.9)
- added SW46: 10u Space, FancyHybridPrints:MX-8U-ReversedStabilizers-NoLED, F.Cu at (190.5, 86.0)
- added SW47: 7u Space, FancyHybridPrints:MX-7U-ReversedStabilizers-NoLED, F.Cu at (190.5, 86.0)
- added SW48: 8, FancyHybridPrints:MX-1U-NoLED, F.Cu at (209.6, 9.75)
- added SW49: I, FancyHybridPrints:MX-1U-NoLED, F.Cu at (219.1, 28.8)
- added SW5: M9, FancyHybridPrints:MX-1U-NoLED, F.Cu at (9.55, 86.0)
- added SW50: J, FancyHybridPrints:MX-1U-NoLED, F.Cu at (204.8, 47.9)
- added SW51: M, FancyHybridPrints:MX-1U-NoLED, F.Cu at (214.3, 66.9)
- added SW52: 9, FancyHybridPrints:MX-1U-NoLED, F.Cu at (228.6, 9.75)
- added SW53: O, FancyHybridPrints:MX-1U-NoLED, F.Cu at (238.2, 28.8)
- added SW54: K, FancyHybridPrints:MX-1U-NoLED, F.Cu at (223.9, 47.9)
- added SW55: ,, FancyHybridPrints:MX-1U-NoLED, F.Cu at (233.4, 66.9)
- added SW56: 0, FancyHybridPrints:MX-1U-NoLED, F.Cu at (247.7, 9.75)
- added SW57: P, FancyHybridPrints:MX-1U-NoLED, F.Cu at (257.2, 28.8)
- added SW58: L, FancyHybridPrints:MX-1U-NoLED, F.Cu at (242.9, 47.9)
- added SW59: ., FancyHybridPrints:MX-1U-NoLED, F.Cu at (252.4, 66.9)
- added SW6: M2, FancyHybridPrints:MX-1U-NoLED, F.Cu at (28.6, 9.75)
- added SW60: -, FancyHybridPrints:MX-1U-NoLED, F.Cu at (266.7, 9.75)
- added SW61: [, FancyHybridPrints:MX-1U-NoLED, F.Cu at (276.2, 28.8)
- added SW62: ;, FancyHybridPrints:MX-1U-NoLED, F.Cu at (262.0, 47.9)
- added SW63: /, FancyHybridPrints:MX-1U-NoLED, F.Cu at (271.5, 66.9)
- added SW64: Alt, FancyHybridPrints:MX-1.5U-NoLED, F.Cu at (281.0, 86.0)
- added SW65: =, FancyHybridPrints:MX-1U-NoLED, F.Cu at (285.8, 9.75)
- added SW66: ], FancyHybridPrints:MX-1U-NoLED, F.Cu at (295.3, 28.8)
- added SW67: ', FancyHybridPrints:MX-1U-NoLED, F.Cu at (281.0, 47.9)
- added SW68: 2.75u Shift, FancyHybridPrints:MX-2.75U-NoLED, F.Cu at (307.2, 66.9)
- added SW69: 1.75u Shift, FancyHybridPrints:MX-1.75U-NoLED, F.Cu at (297.7, 66.9)
- added SW7: M4, FancyHybridPrints:MX-1U-NoLED, F.Cu at (28.6, 28.8)
- added SW70: \, FancyHybridPrints:MX-1U-NoLED, F.Cu at (304.8, 9.75)
- added SW71: 2u Back, FancyHybridPrints:MX-2U-NoLED, F.Cu at (314.4, 9.75)
- added SW72: 1u Back, FancyHybridPrints:MX-1U-NoLED, F.Cu at (323.9, 9.75)
- added SW73: \, FancyHybridPrints:MX-1.5U-NoLED, F.Cu at (319.1, 28.8)
- added SW74: Enter, FancyHybridPrints:MX-2.25U-NoLED, F.Cu at (312.0, 47.9)
- added SW75: Fn, FancyHybridPrints:MX-1U-NoLED, F.Cu at (323.9, 66.9)
- added SW76: Ctrl, FancyHybridPrints:MX-1.5U-NoLED, F.Cu at (319.1, 86.0)
- added SW77: Insert, FancyHybridPrints:MX-1U-NoLED, F.Cu at (352.4, 9.75)
- added SW78: Delete, FancyHybridPrints:MX-1U-NoLED, F.Cu at (352.4, 28.8)
- added SW79: Left, FancyHybridPrints:MX-1U-NoLED, F.Cu at (352.4, 86.0)
- added SW8: M6, FancyHybridPrints:MX-1U-NoLED, F.Cu at (28.6, 47.9)
- added SW80: Home, FancyHybridPrints:MX-1U-NoLED, F.Cu at (371.5, 9.75)
- added SW81: End, FancyHybridPrints:MX-1U-NoLED, F.Cu at (371.5, 28.8)
- added SW82: Up, FancyHybridPrints:MX-1U-NoLED, F.Cu at (371.5, 66.9)
- added SW83: Down, FancyHybridPrints:MX-1U-NoLED, F.Cu at (371.5, 86.0)
- added SW84: PgUp, FancyHybridPrints:MX-1U-NoLED, F.Cu at (390.6, 9.75)
- added SW85: PgDn, FancyHybridPrints:MX-1U-NoLED, F.Cu at (390.6, 28.8)
- added SW86: Right, FancyHybridPrints:MX-1U-NoLED, F.Cu at (390.6, 86.0)
- added SW9: M8, FancyHybridPrints:MX-1U-NoLED, F.Cu at (28.6, 66.9)
- added U1: ATmega32U4-A, keeb:QFN_TQFP-44_Combined, F.Cu at (118.0, 151.6)
- added Y1: Crystal_GND24_Small, keeb:Crystal_SMD_3225-4Pin_3.2x2.5mm_HandSoldering, F.Cu at (122.4, 161.4)

Commit message: placed/routed diodes
Parts:
- D1, D10, D11, D12, D13, D14, D15, D16, D17, D18, D19, D2, D20, D21, D22, D23, D24, D25, D26, D27, D28, D29, D3, D30, D31, D32, D33, D34, D35, D36, D37, D38, D39, D4, D40, D41, D42, D43, D44, D45, D46, D5, D6, D7, D8, D9: moved to B.Cu
- moved D43 353.2 mm to (381.0, 12.8), turned to -90 degrees
- moved D39 342.9 mm to (338.6, 31.8), turned to -90 degrees
- moved D45 339.7 mm to (381.0, 69.9), turned to -90 degrees
- moved D44 338.1 mm to (381.0, 31.8), turned to -90 degrees
- moved D30 334.3 mm to (266.7, 31.8), turned to -90 degrees
- moved D40 332.5 mm to (339.0, 50.9), turned to -90 degrees
- moved D41 323.1 mm to (339.4, 69.9), turned to -90 degrees
- moved D42 317.9 mm to (339.1, 89.0), turned to -90 degrees
- moved D35 309.4 mm to (304.8, 31.8), turned to -90 degrees
- moved D25 307.9 mm to (219.1, 12.8), turned to -90 degrees
- moved D1 300.8 mm to (19.1, 12.8), turned to -90 degrees
- moved D46 300.2 mm to (381.0, 89.0), turned to -90 degrees
- moved D20 291.3 mm to (181.0, 12.8), turned to -90 degrees
- moved D32 289.5 mm to (261.9, 69.9), turned to -90 degrees
- moved D21 286.9 mm to (190.5, 31.8), turned to -90 degrees
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Connections:
- D18 pad 3: Net-(D18-Pad3) -> C3
- D19 pad 3: Net-(D18-Pad3) -> C3
- D28 pad 3: unconnected-(D28-Pad3) -> C5
- SW43 pad 1: R3 -> Net-(D21-Pad2)
- SW43 pad 2: Net-(D21-Pad2) -> R3
Routing:
- net C6: track 0.00 -> 94.2 mm
- net C2: track 0.00 -> 94.0 mm
- net C4: track 0.00 -> 92.1 mm
- net C1: track 0.00 -> 84.1 mm
- net C7: track 0.00 -> 82.8 mm
- net C8: track 0.00 -> 76.7 mm
- net C9: track 0.00 -> 76.2 mm
- net C0: track 0.00 -> 76.2 mm
- net C3: track 0.00 -> 71.1 mm
- net C5: track 0.00 -> 71.0 mm
- net Net-(D37-Pad1): track 0.00 -> 32.0 mm
- net Net-(D8-Pad1): track 0.00 -> 31.3 mm
- net Net-(D40-Pad1): track 0.00 -> 29.1 mm
- net Net-(D38-Pad1): track 0.00 -> 26.9 mm
- net Net-(D42-Pad1): track 0.00 -> 21.8 mm
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
Commit message: routed rows/cols
Parts:
- moved C1 208.2 mm to (137.6, 102.9)
- moved C2 208.2 mm to (155.2, 102.9)
- moved C3 208.2 mm to (168.4, 102.9)
- moved C4 208.2 mm to (142.0, 102.9)
- moved C5 208.2 mm to (146.4, 102.9)
- moved C6 208.2 mm to (150.8, 102.9)
- moved C7 208.2 mm to (128.8, 102.9)
- moved C8 208.2 mm to (164.0, 102.9)
- moved J1 208.2 mm to (118.2, 103.0)
- moved R2 208.2 mm to (124.3, 102.9)
- moved R3 208.2 mm to (159.6, 102.9)
- moved R4 208.2 mm to (133.2, 102.9)
- moved JP1 50.6 mm to (98.9, 112.3)
- moved R1 50.6 mm to (97.0, 115.3)
- moved U1 50.6 mm to (102.0, 103.6)
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Connections:
- SW75 pad 1: Net-(D37-Pad1) -> R6
- SW82 pad 1: Net-(D37-Pad1) -> R6
Routing:
- net R6: track 10.2 -> 473.6 mm
- net R0: track 10.0 -> 459.2 mm
- net R2: track 0.00 -> 445.0 mm
- net R8: track 0.00 -> 398.0 mm
- net R1: track 0.00 -> 394.2 mm
- net R4: track 0.00 -> 382.3 mm
- net R3: track 0.00 -> 381.3 mm
- net R9: track 0.00 -> 368.1 mm
- net R7: track 0.00 -> 259.4 mm
- net R5: track 0.00 -> 245.1 mm
- net Net-(D37-Pad1): track 32.0 -> 20.5 mm
- net Net-(D9-Pad1): track 10.0 -> 20.3 mm

Commit message: placed jst connector
Parts:
- C1, C2, C3, C4, C5, C6, C7, C8, J1, R1, R2, R3, R4, U1, Y1: moved to B.Cu
- moved U1 264.5 mm to (360.6, 48.4), turned to 45 degrees
- moved J1 117.1 mm to (181.0, 4.10)
- moved C3 74.7 mm to (93.8, 102.9), turned to 180 degrees
- moved R1 68.3 mm to (165.2, 115.3), turned to 180 degrees
- moved C8 65.9 mm to (98.2, 102.9), turned to 180 degrees
- moved R3 57.0 mm to (102.6, 102.9), turned to 180 degrees
- moved Y1 49.5 mm to (155.8, 113.5), turned to 180 degrees
- moved C2 48.2 mm to (107.0, 102.9), turned to 180 degrees
- moved JP1 40.3 mm to (139.1, 114.4)
- moved C6 39.4 mm to (111.4, 102.9), turned to 180 degrees
- moved C5 30.6 mm to (115.8, 102.9), turned to 180 degrees
- moved C4 21.8 mm to (120.2, 102.9), turned to 180 degrees
- moved R2 13.5 mm to (137.9, 102.9), turned to 180 degrees
- moved C1 12.9 mm to (124.6, 102.9), turned to 180 degrees
- moved D20 5.00 mm to (176.0, 12.8)
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Routing:
- net Net-(D20-Pad2): track 9.26 -> 14.2 mm
- net Net-(D20-Pad1): track 12.1 -> 7.26 mm
- net C4: track 92.1 -> 95.4 mm
